File: TI Bluetooth.sch (EAGLE design)
At the start: 43 parts, among them J1 DEBUG Connector, J2 USB-C31-S-RA-CS1-BK-TR, J3 Expansion Header, U1 TPS62160, U2 CC2642R1FRGZRRGZ0048A, Y1 32.768kHz, Y2 48MHz

Commit message: Split to two frames
Parts:
- C1: value 10uF -> 1pF
- C10: value 1pF -> 12pF
- C11: value 12pF -> 10uF
- C12: value 1pF -> 22uF
- C13: value 1pF -> 0.1uF
- C15: value 12pF -> 0.1uF
- C16: value 1.8pF -> 22uF
- C2, C5: value 22uF -> 12pF
- C3, C4: value 0.1uF -> 1pF
- C6: value 12pF -> 1.8pF
- J2: value USB-C31-S-RA-CS1-BK-TR -> USB Type C Connector
- L2: value 2.2uH -> 6.8nH
- L6: value 6.8nH -> 2.2uH
- R3: value 562k -> 100k
- R4: value 180k -> 56R
- R5, R6: value 100k -> 56R
- R7: value 56R -> 100k
- R8: value 56R -> 562k
- R9: value 56R -> 180k
Connections:
- removed net 3.3V: ANT1.RETURN, C1.2, C10.2, C11.2, C13.2, C14.2, C2.2, C3.2, C4.2, C5.2, C6.1, C7.1, C8.1, C9.2, R1.2, R4.1, R7.1, R8.1, R9.1, U1.AGND, U1.PGND, U2.EGP
- removed net GND_IN: J2.GND@11, J2.GND@12, J2.GND@21, J2.GND@22
- removed net N$23: J1.GND@3, J1.GND@5
- removed net N$32: J3.2
- removed net N$4: F1.1, R2.1
- new net GND: ANT1.RETURN, C1.2, C10.2, C11.2, C12.2, C13.2, C14.2, C15.2, C16.2, C2.2, C4.2, C7.1, C8.1, C9.1, J1.GND@3, J1.GND@5, J2.GND@11, J2.GND@12, J2.GND@21, J2.GND@22, J3.2, R2.2, R4.1, R5.1, R6.1, R9.1, U1.AGND, U1.PGND, U2.EGP
- net AGND: now also R1.2, R2.1; no longer R1.1, R2.2
- net DCDC_SW_MCU: now also L5.1; no longer L1.1
- net JTAG_RESET_MCU: now also R7.1; no longer R5.1
- net N$1: now also C8.2; no longer C7.2
- net N$10: now also L6.1; no longer L2.1
- net N$12: now also C4.1, L3.2, L4.1; no longer C13.1, L5.2, L6.1
- net N$13: now also C3.2, L2.2, L3.1; no longer C12.2, L4.2, L5.1
- net N$14: now also C5.1, L4.2; no longer C15.1, L6.2
- net N$16: now also R8.1, R9.2; no longer R3.1, R4.2
- net N$17: now also C5.2, C6.1; no longer C15.2, C16.1
- net N$18: now also R4.2; no longer R7.2
- net N$19: now also R6.2; no longer R9.2
- net N$2: now also C9.2; no longer C8.2
- net N$20: now also R5.2; no longer R8.2
- net N$24: now also C6.2; no longer C16.2
- net N$3: now also C10.1; no longer C9.1
- net N$6: now also C2.1, L1.2; no longer C11.1, L3.2
- net N$7: now also C7.2; no longer C6.2
- net POWER_LED: now also R3.1; no longer R6.1
- net RF_N_MCU: now also C1.1, L2.1; no longer C10.1, L4.1
- net RF_P_MCU: now also C3.1, L1.1; no longer C12.1, L3.1
- net V3P3: now also C16.1, L6.2, R7.2, R8.2; no longer C5.1, L2.2, R5.2, R6.2
- net VBUS: now also F1.1, R1.1
- net VBUS_IN: now also C11.1; no longer C1.1
- net VDDR: now also C12.1, C13.1, C15.1, L5.2; no longer C2.1, C3.1, C4.1, L1.2
Other:
- note added: "Expansion Header"
- note added: "LED"
- note removed: "MCU"
- note removed: "USB-A Connector"
- moved on the sheet: C1, C10, C11, C12, C13, C14, C15, C16, C2, C3, C4, C5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

Commit message: Initial routing
Parts:
- D2: value STATUS2 -> STATUS1
- D3: value STATUS1 -> STATUS2
- U2: value CC2642R1FRGZRRGZ0048A -> CC2642R
Connections:
- net GND: no longer R4.1, R5.1, R6.1
- net POWER_LED: now also R4.1; no longer D1.A
- net STATUS1_LED_MCU: now also R5.1, U2.DIO_15; no longer D3.A
- net STATUS2_LED_MCU: now also R6.1, U2.DIO_14; no longer D2.A
- net V3P3: now also D1.A, D2.A, D3.A
Other:
- moved on the sheet: D1, D2, D3, R3, R4, R5, R6

Commit message: Much of routing finished
Connections:
- removed net N$24: ANT1.FEED, C6.2
- net GND: now also ANT1.FEED, C6.2
Changed lines of the file:
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@@
-</segment>
-</net>
-<net name="N$24" class="0">
-<segment>
-<pinref part="C6" gate="G$1" pin="2"/>
-<pinref part="ANT1" gate="ANT_2.4GHZ" pin="FEED"/>
-<wire x1="-205.74" y1="965.2" x2="-215.9" y2="965.2" width="0.1524" layer="91"/>
 </segment>
 </net>
@@
 </segment>
 <segment>
-<pinref part="R4" gate="G$1" pin="1"/>
-<wire x1="-274.32" y1="1018.54" x2="-271.78" y2="1018.54" width="0.1524" layer="91"/>
 <wire x1="-248.92" y1="1018.54" x2="-269.24" y2="1018.54" width="0.1524" layer="91"/>
 <label x="-248.92" y="1018.54" size="1.778" layer="95" align="bottom-right"/>
 <pinref part="R3" gate="G$1" pin="1"/>
-<wire x1="-269.24" y1="1018.54" x2="-274.32" y2="1018.54" width="0.1524" layer="91"/>
 <wire x1="-269.24" y1="1021.08" x2="-269.24" y2="1018.54" width="0.1524" layer="91"/>
+<pinref part="R4" gate="G$1" pin="1"/>
+<wire x1="-274.32" y1="1018.54" x2="-269.24" y2="1018.54" width="0.1524" layer="91"/>
 <junction x="-269.24" y="1018.54"/>
 </segment>
@@
 <pinref part="SUPPLY7" gate="GND" pin="GND"/>
 </segment>
-</net>
+<segment>
+<pinref part="C6" gate="G$1" pin="2"/>
+<pinref part="ANT1" gate="ANT_2.4GHZ" pin="FEED"/>
+<wire x1="-205.74" y1="965.2" x2="-215.9" y2="965.2" width="0.1524" layer="91"/>
+</segment>
+</net>
